Commit message: gazebo_controller

File: urdf/gazebo_control.xacro (robot description, xacro)
@@ -6,6 +6,6 @@
             <left_joint>Revolute 17</left_joint>
             <right_joint>Revolute 16</right_joint>
-            <wheel_separation>0.35</wheel_separation>
-            <wheel_diameter>0.1</wheel_diameter>
+            <wheel_separation>0.194</wheel_separation>
+            <wheel_diameter>0.0425</wheel_diameter>
             <!--Limits-->
             <max_wheel_torque>200</max_wheel_torque>

File: urdf/slambot_core.xacro (robot description, xacro)
@@ -2,7 +2,7 @@
 <robot name="slambot"
   xmlns:xacro="http://www.ros.org/wiki/xacro">
-  <!-- <xacro:macro name="gazebo_description" params="link">
+  <xacro:macro name="gazebo_description" params="link color">
     <gazebo reference="${link}">
-      <material>Gazebo/White</material>
+      <material>${color}</material>
       <mu1>0.2</mu1>
       <mu2>0.2</mu2>
@@ -10,5 +10,5 @@
       <gravity>true</gravity>
     </gazebo>
-  </xacro:macro> -->
+  </xacro:macro>
   <link name="base_link"/>
   <joint name="base_footprint_joint" type="fixed">
@@ -43,5 +43,5 @@
     </collision>
   </link>
-  <!-- <xacro:gazebo_description link="base_plate"/> -->
+  <xacro:gazebo_description link="base_plate" color="Gazebo/White"/>
   <link name="Top2BottomSupport_v1_1">
     <inertial>
@@ -64,5 +64,5 @@
     </collision>
   </link>
-  <!-- <xacro:gazebo_description link="Top2BottomSupport_v1_1"/> -->
+  <xacro:gazebo_description link="Top2BottomSupport_v1_1" color="Gazebo/Black"/>
   <link name="Top2BottomSupport_v1_2">
     <inertial>
@@ -85,5 +85,5 @@
     </collision>
   </link>
-  <!-- <xacro:gazebo_description link="Top2BottomSupport_v1_2"/> -->
+  <xacro:gazebo_description link="Top2BottomSupport_v1_2" color="Gazebo/Black"/>
   <link name="Top2BottomSupport_v1_3">
     <inertial>
@@ -106,5 +106,5 @@
     </collision>
   </link>
-  <!-- <xacro:gazebo_description link="Top2BottomSupport_v1_3"/> -->
+  <xacro:gazebo_description link="Top2BottomSupport_v1_3" color="Gazebo/Black"/>
   <link name="Top2BottomSupport_v1_4">
     <inertial>
@@ -127,5 +127,5 @@
     </collision>
   </link>
-  <!-- <xacro:gazebo_description link="Top2BottomSupport_v1_4"/> -->
+  <xacro:gazebo_description link="Top2BottomSupport_v1_4" color="Gazebo/Black"/>
   <link name="Top_v1_1">
     <inertial>
@@ -148,5 +148,5 @@
     </collision>
   </link>
-  <!-- <xacro:gazebo_description link="Top_v1_1"/> -->
+  <xacro:gazebo_description link="Top_v1_1" color="Gazebo/White"/>
   <link name="20V_Battery_Holder_v1_1">
     <inertial>
@@ -169,5 +169,5 @@
     </collision>
   </link>
-  <!-- <xacro:gazebo_description link="20V_Battery_Holder_v1_1"/> -->
+  <xacro:gazebo_description link="20V_Battery_Holder_v1_1" color="Gazebo/Black"/>
   <link name="Motor_Bracket_v1_1">
     <inertial>
@@ -190,5 +190,5 @@
     </collision>
   </link>
-  <!-- <xacro:gazebo_description link="Motor_Bracket_v1_1"/> -->
+  <xacro:gazebo_description link="Motor_Bracket_v1_1" color="Gazebo/Black"/>
   <link name="Motor_Bracket_v1_2">
     <inertial>
@@ -211,5 +211,5 @@
     </collision>
   </link>
-  <!-- <xacro:gazebo_description link="Motor_Bracket_v1_2"/> -->
+  <xacro:gazebo_description link="Motor_Bracket_v1_2" color="Gazebo/Black"/>
   <link name="Motor_GM25-370_v1_1">
     <inertial>
@@ -232,5 +232,5 @@
     </collision>
   </link>
-  <!-- <xacro:gazebo_description link="Motor_GM25-370_v1_1"/> -->
+  <xacro:gazebo_description link="Motor_GM25-370_v1_1" color="Gazebo/Grey"/>
   <link name="Motor_GM25-370_v1_2">
     <inertial>
@@ -253,5 +253,5 @@
     </collision>
   </link>
-  <!-- <xacro:gazebo_description link="Motor_GM25-370_v1_2"/> -->
+  <xacro:gazebo_description link="Motor_GM25-370_v1_2" color="Gazebo/Grey"/>
   <link name="CastorWheel_Socks_v1_1">
     <inertial>
@@ -274,5 +274,5 @@
     </collision>
   </link>
-  <!-- <xacro:gazebo_description link="CastorWheel_Socks_v1_1"/> -->
+  <xacro:gazebo_description link="CastorWheel_Socks_v1_1" color="Gazebo/Black"/>
   <link name="CastorWheel_Socks_v1_2">
     <inertial>
@@ -295,5 +295,5 @@
     </collision>
   </link>
-  <!-- <xacro:gazebo_description link="CastorWheel_Socks_v1_2"/> -->
+  <xacro:gazebo_description link="CastorWheel_Socks_v1_2" color="Gazebo/Black"/>
   <link name="Caster-swivel-40mmzzzzzzzzz_assembly_v1_1">
     <inertial>
@@ -316,5 +316,5 @@
     </collision>
   </link>
-  <!-- <xacro:gazebo_description link="Caster-swivel-40mmzzzzzzzzz_assembly_v1_1"/> -->
+  <xacro:gazebo_description link="Caster-swivel-40mmzzzzzzzzz_assembly_v1_1" color="Gazebo/Grey"/>
   <link name="Caster-swivel-40mmzzzzzzzzz_assembly_v1_2">
     <inertial>
@@ -337,5 +337,5 @@
     </collision>
   </link>
-  <!-- <xacro:gazebo_description link="Caster-swivel-40mmzzzzzzzzz_assembly_v1_2"/> -->
+  <xacro:gazebo_description link="Caster-swivel-40mmzzzzzzzzz_assembly_v1_2" color="Gazebo/Grey"/>
   <link name="RC_coupling_v1_1">
     <inertial>
@@ -358,5 +358,5 @@
     </collision>
   </link>
-  <!-- <xacro:gazebo_description link="RC_coupling_v1_1"/> -->
+  <xacro:gazebo_description link="RC_coupling_v1_1" color="Gazebo/Black"/>
   <link name="RC_coupling_v1_2">
     <inertial>
@@ -379,5 +379,5 @@
     </collision>
   </link>
-  <!-- <xacro:gazebo_description link="RC_coupling_v1_2"/> -->
+  <xacro:gazebo_description link="RC_coupling_v1_2" color="Gazebo/Black"/>
   <link name="85mm_Wheel_v1_1">
     <inertial>
@@ -400,5 +400,5 @@
     </collision>
   </link>
-  <!-- <xacro:gazebo_description link="85mm_Wheel_v1_1"/> -->
+  <xacro:gazebo_description link="85mm_Wheel_v1_1" color="Gazebo/Black"/>
   <link name="85mm_Wheel_v1_2">
     <inertial>
@@ -421,5 +421,5 @@
     </collision>
   </link>
-  <!-- <xacro:gazebo_description link="85mm_Wheel_v1_2"/> -->
+  <xacro:gazebo_description link="85mm_Wheel_v1_2" color="Gazebo/Black"/>
   <joint name="Rigid 1" type="fixed">
     <origin xyz="-0.061083 -0.088085 0.002998" rpy="0 0 0"/>
@@ -496,5 +496,5 @@
     <parent link="Motor_GM25-370_v1_1"/>
     <child link="RC_coupling_v1_1"/>
-    <axis xyz="1.0 -0.0 0.0"/>
+    <axis xyz="-1.0 -0.0 0.0"/>
   </joint>
   <joint name="Revolute 17" type="continuous">
